File: hardware_package/prototyping/PCB_design/KiCad_files/RocketPCB.sch (KiCad schematic (older format))
At the start: 68 parts

Commit message: Edit slight modifications
Parts:
- removed BT?: Battery_Cell, symbol Device:Battery_Cell
- gave numbers to parts that had none: 67
Connections:
- net labels removed: VBACKUP
- wire segments 324 -> 323
