File: hardware_package/prototyping/PCB_design/full_PCB/RocketPCB.kicad_pcb (KiCad board)
At the start: 2 copper layers, 7 parts, among them J3 Conn_01x03_Female, Q1 DMG2301L, U1 STM32F405RGTx, U2 TPS62160DSG, U6 AP2112K-3.3, U7 MPL3115A2

Commit message: Begun laying out PCB
Parts:
- added C1: 22pF, Capacitor_THT:CP_Radial_D5.0mm_P2.50mm, F.Cu at (225.8, 115.2)
- added C10: 10uF, Capacitor_THT:CP_Radial_D5.0mm_P2.50mm, F.Cu at (125.7, 120.7)
- added C11: 22uF, Capacitor_THT:CP_Radial_D5.0mm_P2.50mm, F.Cu at (158.8, 129.5)
- added C12: 10uF, Capacitor_THT:CP_Radial_D5.0mm_P2.50mm, F.Cu at (239.1, 115.3)
- added C13: 0.1u, Capacitor_THT:CP_Radial_D5.0mm_P2.50mm, F.Cu at (264.5, 91.0)
- added C14: 2.2u, Capacitor_THT:CP_Radial_D5.0mm_P2.50mm, F.Cu at (232.4, 121.7)
- added C15: 10uF, Capacitor_THT:CP_Radial_D5.0mm_P2.50mm, F.Cu at (256.0, 95.6)
- added C16: 10uF, Capacitor_THT:CP_Radial_D5.0mm_P2.50mm, F.Cu at (241.9, 108.7)
- added C17: 1uF, Capacitor_THT:CP_Radial_D5.0mm_P2.50mm, F.Cu at (248.5, 102.2)
- added C18: 100nF, Capacitor_THT:CP_Radial_D5.0mm_P2.50mm, F.Cu at (266.2, 84.5)
- added C19: 1uF, Capacitor_THT:CP_Radial_D5.0mm_P2.50mm, F.Cu at (232.4, 115.1)
- added C2: 22pF, Capacitor_THT:CP_Radial_D5.0mm_P2.50mm, F.Cu at (235.3, 102.0)
- added C20: 10uF, Capacitor_THT:CP_Radial_D5.0mm_P2.50mm, F.Cu at (255.2, 102.2)
- added C21: 1uF, Capacitor_THT:CP_Radial_D5.0mm_P2.50mm, F.Cu at (257.8, 88.5)
- added C22: 10uF, Capacitor_THT:CP_Radial_D5.0mm_P2.50mm, F.Cu at (251.2, 89.1)
- added C23: 1uF, Capacitor_THT:CP_Radial_D5.0mm_P2.50mm, F.Cu at (242.7, 95.6)
- added C24: 100nF, Capacitor_THT:CP_Radial_D5.0mm_P2.50mm, F.Cu at (249.4, 95.6)
- added C25: 1uF, Capacitor_THT:CP_Radial_D5.0mm_P2.50mm, F.Cu at (241.9, 102.2)
- added C26: 1uF, Capacitor_THT:CP_Radial_D5.0mm_P2.50mm, F.Cu at (252.9, 82.0)
- added C27: 1uF, Capacitor_THT:CP_Radial_D5.0mm_P2.50mm, F.Cu at (259.6, 82.0)
- added C28: 10uF, Capacitor_THT:CP_Radial_D5.0mm_P2.50mm, F.Cu at (219.2, 121.8)
- added C29: 0.1uF, Capacitor_THT:CP_Radial_D5.0mm_P2.50mm, F.Cu at (228.6, 108.6)
- added C3: 22pF, Capacitor_THT:CP_Radial_D5.0mm_P2.50mm, F.Cu at (270.0, 71.4)
- added C30: 10pF, Capacitor_THT:CP_Radial_D5.0mm_P2.50mm, F.Cu at (267.2, 77.9)
- added C31: 22uF, Capacitor_THT:CP_Radial_D5.0mm_P2.50mm, F.Cu at (219.2, 115.2)
- added C32: 22uF, Capacitor_THT:CP_Radial_D5.0mm_P2.50mm, F.Cu at (253.9, 75.4)
- added C33: 22uF, Capacitor_THT:CP_Radial_D5.0mm_P2.50mm, F.Cu at (260.5, 74.5)
- added C4: 10uF, Capacitor_THT:CP_Radial_D5.0mm_P2.50mm, F.Cu at (228.6, 102.0)
- added C5: 0.1uF, Capacitor_THT:CP_Radial_D5.0mm_P2.50mm, F.Cu at (244.6, 89.1)
- added C6: 10uF, Capacitor_THT:CP_Radial_D5.0mm_P2.50mm, F.Cu at (239.1, 121.8)
- added C7: 22pF, Capacitor_THT:CP_Radial_D5.0mm_P2.50mm, F.Cu at (235.3, 108.6)
- added C8: 0.1uF, Capacitor_THT:CP_Radial_D5.0mm_P2.50mm, F.Cu at (245.7, 115.3)
- added C9: 10uF, Capacitor_THT:CP_Radial_D5.0mm_P2.50mm, F.Cu at (262.6, 97.6)
- added D1: LED, LED_THT:LED_D5.0mm_Clear, F.Cu at (212.0, 117.6)
- added F1: Polyfuse, Fuse:Fuse_Littelfuse_395Series, F.Cu at (113.0, 110.5)
- added FB1: Ferrite_Bead, Ferrite_THT:LairdTech_28C0236-0JW-10, F.Cu at (233.6, 94.3)
- added J1: USB_C_Receptacle, Connector_USB:USB_C_Receptacle_GCT_USB4085, F.Cu at (190.0, 115.6)
- added J2: Micro_SD_Card, Connector_Card:microSD_HC_Hirose_DM3BT-DSF-PEJS, F.Cu at (194.3, 24.1)
- added L1: 2.2uH, Inductor_THT:L_Axial_L9.5mm_D4.0mm_P12.70mm_Horizontal_Fastron_SMCC, F.Cu at (138.4, 118.1)
- added L2: 1uH, Inductor_THT:L_Axial_L9.5mm_D4.0mm_P12.70mm_Horizontal_Fastron_SMCC, F.Cu at (232.0, 70.9)
- added Q2: Q_PMOS_DGS, Package_TO_SOT_SMD:SOT-23, F.Cu at (101.6, 110.5)
- added R1: 10k, Resistor_THT:R_Axial_DIN0207_L6.3mm_D2.5mm_P7.62mm_Horizontal, F.Cu at (233.3, 83.8)
- added R10: 100k, Resistor_THT:R_Axial_DIN0207_L6.3mm_D2.5mm_P7.62mm_Horizontal, F.Cu at (141.0, 113.0)
- added R11: 649k, Resistor_THT:R_Axial_DIN0207_L6.3mm_D2.5mm_P7.62mm_Horizontal, F.Cu at (151.1, 123.2)
- added R12: 180k, Resistor_THT:R_Axial_DIN0207_L6.3mm_D2.5mm_P7.62mm_Horizontal, F.Cu at (151.1, 133.3)
- added R13: 100k, Resistor_THT:R_Axial_DIN0207_L6.3mm_D2.5mm_P7.62mm_Horizontal, F.Cu at (260.4, 122.9)
- added R14: 1M, Resistor_THT:R_Axial_DIN0204_L3.6mm_D1.6mm_P7.62mm_Horizontal, F.Cu at (200.3, 122.8)
- added R15: 100k, Resistor_THT:R_Axial_DIN0207_L6.3mm_D2.5mm_P7.62mm_Horizontal, F.Cu at (206.6, 103.7)
- added R16: 100k, Resistor_THT:R_Axial_DIN0207_L6.3mm_D2.5mm_P7.62mm_Horizontal, F.Cu at (206.6, 99.6)
- added R19: 10k, Resistor_THT:R_Axial_DIN0207_L6.3mm_D2.5mm_P7.62mm_Horizontal, F.Cu at (231.8, 79.7)
- added R2: 5.1k, Resistor_THT:R_Axial_DIN0207_L6.3mm_D2.5mm_P7.62mm_Horizontal, F.Cu at (233.3, 87.8)
- added R3: 5.1k, Resistor_THT:R_Axial_DIN0207_L6.3mm_D2.5mm_P7.62mm_Horizontal, F.Cu at (242.6, 75.7)
- added R4: 100k, Resistor_THT:R_Axial_DIN0207_L6.3mm_D2.5mm_P7.62mm_Horizontal, F.Cu at (217.3, 104.4)
- added R5: 2.2k, Resistor_THT:R_Axial_DIN0207_L6.3mm_D2.5mm_P7.62mm_Horizontal, F.Cu at (206.6, 111.8)
- added R6: 100k, Resistor_THT:R_Axial_DIN0207_L6.3mm_D2.5mm_P7.62mm_Horizontal, F.Cu at (217.3, 100.3)
- added R7: 100k, Resistor_THT:R_Axial_DIN0207_L6.3mm_D2.5mm_P7.62mm_Horizontal, F.Cu at (206.6, 107.7)
- added R8: 2.2M, Resistor_THT:R_Axial_DIN0204_L3.6mm_D1.6mm_P7.62mm_Horizontal, F.Cu at (200.3, 119.7)
- added R9: 200k, Resistor_THT:R_Axial_DIN0204_L3.6mm_D1.6mm_P7.62mm_Horizontal, F.Cu at (258.7, 69.7)
- added SW1: SW_Push, Button_Switch_THT:SW_PUSH-12mm, F.Cu at (167.6, 71.1)
- added SW2: SW_Push, Button_Switch_THT:SW_PUSH-12mm, F.Cu at (162.6, 3.81)
- added U3: Radio_Header, GPS_head0:gps_header_footprint, F.Cu at (189.2, 85.1)
- added U4: MPU-6050, GPS_head0:MPU6050-footprint, F.Cu at (194.0, 98.8)
- added U5: W25Q16JV, GPS_head0:W25Q16JV_footprint, F.Cu at (246.0, 85.0)
- added U8: GPS_header, GPS_head0:GPS_header_fp, F.Cu at (220.1, 83.3)
- added U9: TPS63060, Package_SON:Texas_S-PWSON-N10_ThermalVias, F.Cu at (125.7, 82.5)
- added Y1: 12MHz, Oscillator:Oscillator_DIP-14_LargePads, F.Cu at (232.4, 7.62)
- added Y2: 32MHz, Oscillator:Oscillator_DIP-8_LargePads, F.Cu at (215.9, 61.0)
- moved U7 172.2 mm to (289.6, 76.2)
- moved J3 130.9 mm to (92.7, 115.6), turned to 90 degrees
- moved U6 101.2 mm to (295.9, 97.8)
- moved U2 93.4 mm to (133.0, 117.9)
- moved Q1 75.6 mm to (280.7, 61.0)
- moved U1 73.1 mm to (193.0, 55.9)
- moved D3 29.8 mm to (212.2, 123.0)
Connections:
- net TP3 renamed +BATT
- J3 pad 3: +7.5V -> Net-(J3-Pad3)
- U1 pad 14: Net-(U1-Pad14) -> /RXI
- U1 pad 15: Net-(U1-Pad15) -> /TX0
- U1 pad 16: Net-(U1-Pad16) -> /PPS
- U1 pad 41: Net-(U1-Pad41) -> /G0
- U1 pad 50: /FLASH_CS -> +3V3
