File: hardware_package/avionics_pcb/full_PCB/RocketPCB.sch (KiCad schematic (older format))
At the start: 72 parts, among them J1 DX07S024XJ1R1100, J2 Micro_SD_Card, J3 Conn_01x03_Female, M1 Motor_Servo_JR, M2 Motor_Servo_JR, Q1 DMG2301L, Q2 DMG2301L, SW1 SW_Push, SW2 SW_Push, U1 STM32F405RGTx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

Commit message: Modified to 4 layer PCB, laid out 6V and 3V3 regulators
Parts:
- added R?: 4.7K, Resistor_SMD:R_0603_1608Metric, symbol Device:R
- C7: value C -> 100nF
Connections:
- net labels removed: A0, CLKIN, CS, FSYNC_IN, INT, INT1, INT2, PPS
- wire segments 360 -> 364
- no-connect marks 42 -> 51
Changed lines of the file:
@@
 Text Label 5850 2200 0    50   ~ 0
 BOOT0
-Text Label 7650 2400 0    50   ~ 0
-A0
-Text Label 7650 2500 0    50   ~ 0
-INT2
-Text Label 7650 2600 0    50   ~ 0
-INT1
 Text Notes 7950 2450 0    50   ~ 0
 DACs
@@
 Wire Wire Line
 	7550 4700 8000 4700
-$Comp
-L MCU_ST_STM32F4:STM32F405RGTx U1
-U 1 1 5F2C61AB
-P 6850 3600
-F 0 "U1" H 6450 1850 50  0000 C CNN
-F 1 "STM32F405RGTx" H 6800 3700 50  0000 C CNN
-F 2 "Package_QFP:LQFP-64_10x10mm_P0.5mm" H 6250 1900 50  0001 R CNN
-F 3 "http://www.st.com/st-web-ui/static/active/en/resource/technical/document/datasheet/DM00037051.pdf" H 6850 3600 50  0001 C CNN
-	1    6850 3600
-	1    0    0    -1
-$EndComp
 Wire Wire Line
 	7650 3000 7550 3000
@@
 FLASH_MOSI
 Wire Wire Line
-	8600 4050 8600 4200
-Wire Wire Line
 	8450 4200 8600 4200
 $Comp
@@
 Wire Wire Line
 	7650 2900 7650 3000
-Text Label 7650 2700 0    50   ~ 0
-INT
 Wire Wire Line
 	6850 5500 6950 5500
@@
 Wire Notes Line
 	11800 9950 11800 8050
-Text Label 10250 1900 0    59   ~ 0
-INT
-Text Label 11950 1500 0    59   ~ 0
-FSYNC_IN
-Text Label 11900 1800 0    59   ~ 0
-CLKIN
 Text Label 10000 1700 0    59   ~ 0
 SCL
@@
 Wire Wire Line
 	7550 3700 8000 3700
-Text Label 7750 3700 0    50   ~ 0
-CS
 $Comp
 L power:GND #PWR030
@@
 Wire Wire Line
 	14800 6400 15250 6400
-Text Label 14900 6300 0    71   ~ 0
-INT1
-Text Label 14900 6400 0    71   ~ 0
-INT2
 Text Notes 12750 5150 0    71   ~ 0
 Barometer\n
@@
 Wire Wire Line
 	10400 4650 9700 4650
-Wire Wire Line
-	10400 4750 9700 4750
 $Comp
 L power:GND #PWR0102
@@
 Wire Wire Line
 	7550 2200 7850 2200
-Text Label 7650 2200 0    47   ~ 0
-PPS
-Text Label 14650 8800 0    47   ~ 0
-PPS
 Text Label 14700 9000 0    47   ~ 0
 RX_D0
@@
 Wire Wire Line
 	7550 2800 7850 2800
-Text Label 7650 2800 0    47   ~ 0
-G0
-Text Label 9900 4250 0    47   ~ 0
-G0
 Text Label 9900 4350 0    47   ~ 0
 SCK
@@
 Text Label 9900 4550 0    47   ~ 0
 MOSI
-Text Label 9900 4650 0    47   ~ 0
-CS
 Text Notes 11900 8200 0    71   ~ 0
 GPS Module
@@
 	1    0    0    -1
 $EndComp
-Wire Wire Line
-	7550 2000 7850 2000
 Wire Wire Line
 	7550 2100 7850 2100
@@
 Text GLabel 12550 9200 0    47   Output ~ 0
 ~RESET~
-Text GLabel 9700 4750 0    47   Input ~ 0
+Text GLabel 10100 4750 0    47   Input ~ 0
 ~RESET~
 NoConn ~ 7800 3500
@@
 P 850 10400
 F 0 "C7" H 965 10446 50  0000 L CNN
-F 1 "C" H 965 10355 50  0000 L CNN
+F 1 "100nF" H 965 10355 50  0000 L CNN
 F 2 "Capacitor_SMD:C_0603_1608Metric" H 888 10250 50  0001 C CNN
 F 3 "~" H 850 10400 50  0001 C CNN
@@
 NoConn ~ 1200 1900
 NoConn ~ 1200 1800
+Wire Wire Line
+	8600 4050 8600 4200
+Wire Wire Line
+	7550 2000 7850 2000
+$Comp
+L MCU_ST_STM32F4:STM32F405RGTx U1
+U 1 1 5F2C61AB
+P 6850 3600
+F 0 "U1" H 6450 1850 50  0000 C CNN
+F 1 "STM32F405RGTx" H 6800 3700 50  0000 C CNN
+F 2 "Package_QFP:LQFP-64_10x10mm_P0.5mm" H 6250 1900 50  0001 R CNN
+F 3 "http://www.st.com/st-web-ui/static/active/en/resource/technical/document/datasheet/DM00037051.pdf" H 6850 3600 50  0001 C CNN
+	1    6850 3600
+	1    0    0    -1
+$EndComp
+NoConn ~ 10150 1900
+$Comp
+L Device:R R?
+U 1 1 608B0935
+P 9550 4650
+F 0 "R?" H 9620 4696 50  0000 L CNN
+F 1 "4.7K" H 9620 4605 50  0000 L CNN
+F 2 "Resistor_SMD:R_0603_1608Metric" V 9480 4650 50  0001 C CNN
+F 3 "~" H 9550 4650 50  0001 C CNN
+	1    9550 4650
+	0    -1   -1   0
+$EndComp
+Wire Wire Line
+	10100 4750 10400 4750
+Wire Wire Line
+	9400 4650 9350 4650
+Wire Wire Line
+	9350 4650 9350 4700
+Text GLabel 9400 4750 3    47   Output ~ 0
++3V3
+NoConn ~ 8000 3700
+NoConn ~ 7850 2700
+Wire Wire Line
+	9400 4750 9400 4700
+Wire Wire Line
+	9400 4700 9350 4700
+NoConn ~ 7850 2200
+NoConn ~ 14950 8800
+Text Label 7650 2800 0    47   ~ 0
+G0
+Text Label 9900 4250 0    47   ~ 0
+G0
+NoConn ~ 15250 6300
+NoConn ~ 15250 6400
+NoConn ~ 7850 2500
+NoConn ~ 7850 2600
 $EndSCHEMATC

Commit message: Laid out and routed the majority of the board
Parts:
- removed TP1: TestPoint, TestPoint:TestPoint_Pad_D1.0mm, symbol Connector:TestPoint
- FB1: footprint Ferrite_THT:LairdTech_28C0236-0JW-10 -> Resistor_SMD:R_0402_1005Metric
- J1: footprint JAE_DX07S024XJ1R1100 -> DX07S024XJ1R1100:JAE_DX07S024XJ1R1100
- gave numbers to parts that had none: 1
Connections:
- wire segments 364 -> 363
- no-connect marks 51 -> 53
Changed lines of the file:
@@
 F 0 "FB1" V 7776 1000 50  0000 C CNN
 F 1 "Ferrite_Bead" V 7867 1000 50  0000 C CNN
-F 2 "Ferrite_THT:LairdTech_28C0236-0JW-10" V 7980 1000 50  0001 C CNN
+F 2 "Resistor_SMD:R_0402_1005Metric" V 7980 1000 50  0001 C CNN
 F 3 "~" H 8050 1000 50  0001 C CNN
 	1    8050 1000
@@
 SDIO_D2
 Text Label 6150 4600 2    50   ~ 0
+SDIO_D0
+Text Label 6150 4500 2    50   ~ 0
 SDIO_D1
-Text Label 6150 4500 2    50   ~ 0
-SDIO_D0
 Text Label 6000 4400 2    50   ~ 0
 D5
@@
 Text Notes 2500 3950 0    71   ~ 0
 Reset & Prog Switches\n
-Wire Wire Line
-	6650 1250 6650 1800
 Text Notes 7600 8200 0    71   ~ 0
 Battery Regulator\n
@@
 Wire Wire Line
 	5650 2500 6150 2500
-$Comp
-L Connector:TestPoint TP1
-U 1 1 60517AA2
-P 6650 1250
-F 0 "TP1" H 6708 1368 50  0000 L CNN
-F 1 "TestPoint" H 6708 1277 50  0000 L CNN
-F 2 "TestPoint:TestPoint_Pad_D1.0mm" H 6850 1250 50  0001 C CNN
-F 3 "~" H 6850 1250 50  0001 C CNN
-	1    6650 1250
-	1    0    0    -1
-$EndComp
 NoConn ~ 7850 2400
 Wire Wire Line
@@
 F 0 "J1" H 2150 2965 50  0000 C CNN
 F 1 "DX07S024XJ1R1100" H 2150 2874 50  0000 C CNN
-F 2 "JAE_DX07S024XJ1R1100" H 2150 2000 50  0001 L BNN
+F 2 "DX07S024XJ1R1100:JAE_DX07S024XJ1R1100" H 2150 2000 50  0001 L BNN
 F 3 "JAE" H 2150 2000 50  0001 L BNN
 F 4 "3.34mm" H 2150 2000 50  0001 L BNN "Field4"
@@
 NoConn ~ 10150 1900
 $Comp
-L Device:R R?
+L Device:R R16
 U 1 1 608B0935
 P 9550 4650
-F 0 "R?" H 9620 4696 50  0000 L CNN
+F 0 "R16" H 9620 4696 50  0000 L CNN
 F 1 "4.7K" H 9620 4605 50  0000 L CNN
 F 2 "Resistor_SMD:R_0603_1608Metric" V 9480 4650 50  0001 C CNN
@@
 NoConn ~ 7850 2500
 NoConn ~ 7850 2600
+NoConn ~ 6650 1800
+NoConn ~ 5200 2750
 $EndSCHEMATC

Commit message: Updated with the correct version
Parts:
- removed J1: DX07S024XJ1R1100, DX07S024XJ1R1100:JAE_DX07S024XJ1R1100, symbol USB-C_symbol:DX07S024XJ1R1100
- added J1: USB_C_Receptacle, Connector_USB:USB_C_Receptacle_Palconn_UTC16-G, symbol Connector:USB_C_Receptacle
Connections:
- wire segments 363 -> 370
- no-connect marks 53 -> 54
Changed lines of the file:
@@
 	3850 6450 9300 6450
-Wire Notes Line
-	500  3800 3850 3800
 Wire Notes Line
 	9300 3150 12650 3150
@@
 NoConn ~ 12250 1400
 NoConn ~ 12200 1800
-$Comp
-L USB-C_symbol:DX07S024XJ1R1100 J1
-U 1 1 600603B9
-P 2150 2000
-F 0 "J1" H 2150 2965 50  0000 C CNN
-F 1 "DX07S024XJ1R1100" H 2150 2874 50  0000 C CNN
-F 2 "DX07S024XJ1R1100:JAE_DX07S024XJ1R1100" H 2150 2000 50  0001 L BNN
-F 3 "JAE" H 2150 2000 50  0001 L BNN
-F 4 "3.34mm" H 2150 2000 50  0001 L BNN "Field4"
-F 5 "1" H 2150 2000 50  0001 L BNN "Field5"
-F 6 "Manufacturer recommendations" H 2150 2000 50  0001 L BNN "Field6"
-	1    2150 2000
-	1    0    0    -1
-$EndComp
-Text Label 3050 1600 2    50   ~ 0
-D-
-Text Label 1400 1600 2    50   ~ 0
-D-
-Text Label 3050 1500 2    50   ~ 0
-D+
-Text Label 1400 1500 2    50   ~ 0
-D+
-$Comp
-L power:GND #PWR011
-U 1 1 60097787
-P 3500 2400
-F 0 "#PWR011" H 3500 2150 50  0001 C CNN
-F 1 "GND" H 3505 2227 50  0000 C CNN
-F 2 "" H 3500 2400 50  0001 C CNN
-F 3 "" H 3500 2400 50  0001 C CNN
-	1    3500 2400
-	0    -1   -1   0
-$EndComp
-$Comp
-L Device:R R2
-U 1 1 60099F83
-P 1050 2400
-F 0 "R2" H 980 2354 50  0000 R CNN
-F 1 "5.1k" H 980 2445 50  0000 R CNN
-F 2 "Resistor_SMD:R_0603_1608Metric" V 980 2400 50  0001 C CNN
-F 3 "~" H 1050 2400 50  0001 C CNN
-	1    1050 2400
-	0    -1   -1   0
-$EndComp
-$Comp
-L Device:R R3
-U 1 1 6009A378
-P 3150 2400
-F 0 "R3" H 3080 2354 50  0000 R CNN
-F 1 "5.1k" H 3080 2445 50  0000 R CNN
-F 2 "Resistor_SMD:R_0603_1608Metric" V 3080 2400 50  0001 C CNN
-F 3 "~" H 3150 2400 50  0001 C CNN
-	1    3150 2400
-	0    1    1    0
-$EndComp
-Text GLabel 3200 1300 2    47   Input ~ 0
-VBUS
-$Comp
-L power:GND #PWR09
-U 1 1 6009C4EA
-P 3150 2600
-F 0 "#PWR09" H 3150 2350 50  0001 C CNN
-F 1 "GND" H 3155 2427 50  0000 C CNN
-F 2 "" H 3150 2600 50  0001 C CNN
-F 3 "" H 3150 2600 50  0001 C CNN
-	1    3150 2600
-	0    -1   -1   0
-$EndComp
-Wire Wire Line
-	1450 1600 1200 1600
-Wire Wire Line
-	2850 1600 3150 1600
-Wire Wire Line
-	2850 1500 3150 1500
-Wire Wire Line
-	1450 1500 1200 1500
-Wire Wire Line
-	2850 1300 3200 1300
-Wire Wire Line
-	2850 2600 3150 2600
-Wire Wire Line
-	2850 2400 3000 2400
-Wire Wire Line
-	3300 2400 3500 2400
-Wire Wire Line
-	1450 2400 1200 2400
-$Comp
-L power:GND #PWR07
-U 1 1 60238A05
-P 700 2400
-F 0 "#PWR07" H 700 2150 50  0001 C CNN
-F 1 "GND" H 705 2227 50  0000 C CNN
-F 2 "" H 700 2400 50  0001 C CNN
-F 3 "" H 700 2400 50  0001 C CNN
-	1    700  2400
-	0    1    1    0
-$EndComp
-Wire Wire Line
-	900  2400 700  2400
-Wire Wire Line
-	2850 2300 2950 2300
-Wire Wire Line
-	2850 2100 3150 2100
-Wire Wire Line
-	2850 2000 3150 2000
-Wire Wire Line
-	2850 1900 3150 1900
-Wire Wire Line
-	2850 1800 3150 1800
-NoConn ~ 2950 2300
-NoConn ~ 3150 2100
-NoConn ~ 3150 2000
-NoConn ~ 3150 1900
-NoConn ~ 3150 1800
-Wire Wire Line
-	1450 2300 1200 2300
-Wire Wire Line
-	1450 2100 1200 2100
-Wire Wire Line
-	1450 2000 1200 2000
-Wire Wire Line
-	1450 1900 1200 1900
-Wire Wire Line
-	1450 1800 1200 1800
-NoConn ~ 1200 2300
-NoConn ~ 1200 2100
-NoConn ~ 1200 2000
-NoConn ~ 1200 1900
-NoConn ~ 1200 1800
 Wire Wire Line
 	8600 4050 8600 4200
@@
 NoConn ~ 6650 1800
 NoConn ~ 5200 2750
+NoConn ~ 2100 3100
+NoConn ~ 2100 3000
+NoConn ~ 2100 2800
+NoConn ~ 2100 2700
+NoConn ~ 2100 2500
+NoConn ~ 2100 2400
+NoConn ~ 2100 2200
+NoConn ~ 2100 2100
+NoConn ~ 2100 1900
+NoConn ~ 2100 1800
+Wire Wire Line
+	2000 1500 2350 1500
+Wire Wire Line
+	2600 1000 2650 1000
+Connection ~ 2600 1000
+Wire Wire Line
+	2600 1100 2600 1000
+Wire Wire Line
+	2500 1100 2600 1100
+Wire Wire Line
+	2500 1000 2600 1000
+$Comp
+L power:GND #PWR09
+U 1 1 5FD05A10
+P 2650 1000
+F 0 "#PWR09" H 2650 750 50  0001 C CNN
+F 1 "GND" H 2655 827 50  0000 C CNN
+F 2 "" H 2650 1000 50  0001 C CNN
+F 3 "" H 2650 1000 50  0001 C CNN
+	1    2650 1000
+	0    -1   -1   0
+$EndComp
+Wire Wire Line
+	1900 1100 2200 1100
+Wire Wire Line
+	1900 1000 2200 1000
+$Comp
+L Connector:USB_C_Receptacle J1
+U 1 1 5F882D78
+P 1300 1800
+F 0 "J1" H 1407 3067 50  0000 C CNN
+F 1 "USB_C_Receptacle" H 1407 2976 50  0000 C CNN
+F 2 "Connector_USB:USB_C_Receptacle_Palconn_UTC16-G" H 1450 1800 50  0001 C CNN
+F 3 "https://www.usb.org/sites/default/files/documents/usb_type-c.zip" H 1450 1800 50  0001 C CNN
+	1    1300 1800
+	1    0    0    -1
+$EndComp
+$Comp
+L Device:R R3
+U 1 1 5FC3CEF9
+P 2350 1100
+F 0 "R3" H 2280 1054 50  0000 R CNN
+F 1 "5.1k" H 2280 1145 50  0000 R CNN
+F 2 "Resistor_SMD:R_0603_1608Metric" V 2280 1100 50  0001 C CNN
+F 3 "~" H 2350 1100 50  0001 C CNN
+	1    2350 1100
+	0    -1   -1   0
+$EndComp
+$Comp
+L Device:R R2
+U 1 1 5FC3C7BA
+P 2350 1000
+F 0 "R2" H 2280 954 50  0000 R CNN
+F 1 "5.1k" H 2280 1045 50  0000 R CNN
+F 2 "Resistor_SMD:R_0603_1608Metric" V 2280 1000 50  0001 C CNN
+F 3 "~" H 2350 1000 50  0001 C CNN
+	1    2350 1000
+	0    1    1    0
+$EndComp
+NoConn ~ 1000 3600
+$Comp
+L power:GND #PWR07
+U 1 1 5FC072E4
+P 1300 3600
+F 0 "#PWR07" H 1300 3350 50  0001 C CNN
+F 1 "GND" H 1305 3427 50  0000 C CNN
+F 2 "" H 1300 3600 50  0001 C CNN
+F 3 "" H 1300 3600 50  0001 C CNN
+	1    1300 3600
+	1    0    0    -1
+$EndComp
+Wire Wire Line
+	1000 3400 1000 3600
+Wire Wire Line
+	1300 3400 1300 3600
+Wire Wire Line
+	1900 3100 2100 3100
+Wire Wire Line
+	1900 3000 2100 3000
+Wire Wire Line
+	1900 2800 2100 2800
+Wire Wire Line
+	1900 2700 2100 2700
+Wire Wire Line
+	1900 2500 2100 2500
+Wire Wire Line
+	1900 2400 2100 2400
+Wire Wire Line
+	1900 2200 2100 2200
+Wire Wire Line
+	1900 2100 2100 2100
+Wire Wire Line
+	1900 1900 2100 1900
+Wire Wire Line
+	1900 1800 2100 1800
+Connection ~ 2000 1500
+Wire Wire Line
+	2000 1600 2000 1500
+Wire Wire Line
+	1900 1600 2000 1600
+Wire Wire Line
+	1900 1500 2000 1500
+Text Label 2350 1500 2    50   ~ 0
+D+
+Connection ~ 2000 1300
+Wire Wire Line
+	1900 1300 2000 1300
+Wire Wire Line
+	2000 1300 2350 1300
+Wire Wire Line
+	2000 1400 2000 1300
+Wire Wire Line
+	1900 1400 2000 1400
+Text Label 2350 1300 2    50   ~ 0
+D-
+Wire Wire Line
+	1900 800  2350 800
+Text GLabel 2350 800  2    47   Input ~ 0
+VBUS
+Wire Notes Line
+	500  3800 3850 3800
 $EndSCHEMATC
